Commit message: velodyne parent frame is now base, not the camera. Biggest change in this commit is that frame change. Adding a rviz config.

File: laikago_ros/laikago_description/xacro/robot.xacro (robot description, xacro)
@@ -138,6 +138,6 @@
     <link name="camera_rgb_optical_frame"/>
     <xacro:include filename="$(find velodyne_description)/urdf/VLP-16.urdf.xacro"/>
-    <VLP-16 parent="camera_link" name="velodyne" topic="lidar_points" hz="10" samples="1024" gpu="false" lasers="16" max_range="100">
-        <origin xyz="0 0.05 0.00" rpy="0 0 0" />
+    <VLP-16 parent="base" name="velodyne" topic="lidar_points" hz="10" samples="1024" gpu="false" lasers="16" max_range="100">
+        <origin xyz="0 0.0 0.11" rpy="0 0 0" />
     </VLP-16>
     <xacro:leg name="FR" mirror="-1" mirror_dae="False" front_hind="1" front_hind_dae="True">
