Commit message: localization fixed

File: laikago_ros/laikago_gazebo/launch/gazebo.xacro (robot description, xacro)
@@ -99,9 +99,29 @@
     </sensor>
   </gazebo>
+ <gazebo>
+      <plugin name="force_based_move_controller" filename="libgazebo_ros_force_based_move.so">
+        <commandTopic>/cmd_vel_raw</commandTopic>
+        <odometryTopic>odom</odometryTopic>
+        <odometryFrame>odom</odometryFrame>
+        <odometryRate>20.0</odometryRate>
+        <robotBaseFrame>base</robotBaseFrame>
+        <yaw_velocity_p_gain>250</yaw_velocity_p_gain>
+        <publishOdometryTf>1</publishOdometryTf>
+      </plugin>
+    </gazebo>
+    <!--<plugin name="p3d_base_controller" filename="libgazebo_ros_p3d.so">-->
+      <!--<alwaysOn>true</alwaysOn>-->
+      <!--<updateRate>50.0</updateRate>-->
+      <!--<bodyName>base</bodyName>-->
+      <!--<topicName>ground_truth/state</topicName>-->
+      <!--<gaussianNoise>0.01</gaussianNoise>-->
+      <!--<frameName>world</frameName>-->
+      <!--<xyzOffsets>0 0 0</xyzOffsets>-->
+      <!--<rpyOffsets>0 0 0</rpyOffsets>-->
+    <!--</plugin>-->
   <gazebo>
     <plugin name="diff_drive_controller" filename="libgazebo_ros_diff_drive.so">
       <publishWheelTF>true</publishWheelTF>
       <publishOdomTF>true</publishOdomTF>
-      <!-- <broadcastTF>true</broadcastTF> -->
       <alwaysOn>true</alwaysOn>
       <legacyMode>false</legacyMode>
@@ -204,4 +224,36 @@
         <material>Gazebo/Red</material>
     </gazebo>
+    <!--<gazebo reference="camera_link">-->
+        <!--<material>Gazebo/FlatBlack</material>-->
+    <!--<sensor type="gpu_ray" name="lds_lfcd_sensor">-->
+      <!--<pose>0 0 0.3 0 0 0</pose>-->
+      <!--<visualize>true</visualize>-->
+      <!--<update_rate>5</update_rate>-->
+      <!--<ray>-->
+        <!--<scan>-->
+          <!--<horizontal>-->
+            <!--<samples>360</samples>-->
+            <!--<resolution>1</resolution>-->
+            <!--<min_angle>0.0</min_angle>-->
+            <!--<max_angle>6.28319</max_angle>-->
+          <!--</horizontal>-->
+        <!--</scan>-->
+        <!--<range>-->
+          <!--<min>0.120</min>-->
+          <!--<max>10.0</max>-->
+          <!--<resolution>0.015</resolution>-->
+        <!--</range>-->
+        <!--<noise>-->
+          <!--<type>gaussian</type>-->
+          <!--<mean>0.0</mean>-->
+          <!--<stddev>0.01</stddev>-->
+        <!--</noise>-->
+      <!--</ray>-->
+      <!--<plugin name="gazebo_ros_lds_lfcd_controller" filename="libgazebo_ros_gpu_laser.so">-->
+        <!--<topicName>scan</topicName>-->
+        <!--<frameName>camera_link</frameName>-->
+      <!--</plugin>-->
+    <!--</sensor>-->
+  <!--</gazebo>-->
     <!-- FL leg -->
     <gazebo reference="FL_hip">
